Commit message: 增加机械臂扫查功能

File: src/aubo_description/urdf/aubo_i5.urdf (robot description, URDF)
Before this commit: robot aubo_i5, 8 links, 7 joints
Joints:
- joint upperArm_joint: limit lower=-3.05 upper=3.05 effort=0 velocity=0 -> lower=-1.57 upper=1.57 effort=0 velocity=0

File: src/aubo_description/urdf/aubo_i5.urdf.xacro (robot description, xacro)
@@ -86,5 +86,5 @@
     <child link="upperArm_Link" />
     <axis xyz="0 0 1" />
-    <limit lower="-3.05" upper="3.05" effort="0" velocity="0" />
+    <limit lower="-1.57" upper="1.57" effort="0" velocity="0" />
   </joint>
   <link name="foreArm_Link">

File: src/aubo_gazebo/urdf/aubo_i5.xacro (robot description, xacro)
@@ -165,5 +165,5 @@
     <child link="upperArm_Link" />
     <axis xyz="0 0 1" />
-    <limit lower="-3.05" upper="3.05" effort="300" velocity="100" />
+    <limit lower="-1.57" upper="1.57" effort="300" velocity="100" />
   </joint>
   <!--/////////////////////////////// FOREARM_LINK ////////////////////////////////////-->
