Commit message: 实现坐标系转换

File: src/aubo_description/urdf/aubo_i5_robot.urdf.xacro (robot description, xacro)
@@ -11,5 +11,5 @@
   <joint name="world_joint" type="fixed">
     <parent link="world" />
-    <child link = "base_link" />
+    <child link="base_link" />
     <origin xyz="0.0 0.0 0.0" rpy="0.0 0.0 0.0" />
   </joint>
